File: Line Follower Sensor/Modulo IR.sch (KiCad schematic (older format))
At the start: 10 parts, among them U1 LM358N, U10 100nF, U12 TCRT5000, U13 100R, U3 1K, U5 20K, U6 10K, U7 POT, U8 CON3_ET, U9 LED

Commit message: Esquema corregido y ERC pasado
Parts:
- U7: symbol POT -> POT-RESCUE-Modulo_IR
- U9: symbol LED -> LED-RESCUE-Modulo_IR
Changed lines of the file:
@@
 EESchema Schematic File Version 2
+LIBS:Modulo IR-rescue
 LIBS:power
 LIBS:device
@@
 encoding utf-8
 Sheet 1 1
-Title ""
+Title "Line Follower Sensor"
 Date ""
-Rev ""
-Comp ""
-Comment1 ""
+Rev "V1.0"
+Comp "Frizzy Electronics"
+Comment1 "Ionut Morariu"
 Comment2 ""
 Comment3 ""
@@
 $EndComp
 $Comp
-L POT U7
+L POT-RESCUE-Modulo_IR U7
 U 1 1 5815DD66
 P 6000 2800
@@
 $EndComp
 $Comp
-L LED U9
+L LED-RESCUE-Modulo_IR U9
 U 1 1 5815EB38
 P 7950 3200

Commit message: Modelos 3D añadidos
Parts:
- U7: value POT -> 10k
Changed lines of the file:
@@
 P 6000 2800
 F 0 "U7" H 6000 2700 50  0000 C CNN
-F 1 "POT" H 6000 2800 50  0000 C CNN
+F 1 "10k" H 6000 2800 50  0000 C CNN
 F 2 "Potentiometers:Potentiometer_Trimmer-Suntan-TSR-3386P" H 6000 2800 50  0001 C CNN
 F 3 "" H 6000 2800 50  0000 C CNN

Commit message: Serigrafia realizada y placa mandada a fabrica
Parts:
- U8: footprint Connectors_JST:JST_XH_S03B-XH-A_03x2.50mm_Angled -> Connectors_JST:JST_PH_S3B-PH-K_03x2.00mm_Angled
Changed lines of the file:
@@
 F 0 "U8" H 9200 4250 50  0000 C CNN
 F 1 "CON3_ET" V 9300 4050 50  0000 C CNN
-F 2 "Connectors_JST:JST_XH_S03B-XH-A_03x2.50mm_Angled" H 9200 4050 50  0001 C CNN
+F 2 "Connectors_JST:JST_PH_S3B-PH-K_03x2.00mm_Angled" H 9200 4050 50  0001 C CNN
 F 3 "" H 9200 4050 50  0000 C CNN
 	1    9200 4050
