File: Modulo IR.sch (KiCad schematic (older format))
At the start: 10 parts, among them U1 LM358N, U10 100nF, U12 TCRT5000, U13 100R, U3 1K, U5 20K, U6 10K, U7 10k, U8 CON3_ET, U9 LED

Commit message: arbol de carpetas cambiado
Parts:
- U1: footprint SMD_Packages:SOIC-8-N -> lib_fp:SOIC-8-N
- U10, U13, U3, U5, U6: footprint Resistors_SMD:R_0805 -> lib_fp:R_0805
- U12: footprint cyclophone:TCRT5000 -> lib_fp:TCRT5000
- U7: footprint Potentiometers:Potentiometer_Trimmer_Bourns_3296W -> lib_fp:Potentiometer_Trimmer_Bourns_3296W
- U8: footprint Connectors_JST:JST_PH_S3B-PH-K_03x2.00mm_Angled -> lib_fp:JST_PH_S3B-PH-K_03x2.00mm_Angled
- U9: footprint LEDs:LED_0805 -> lib_fp:LED_0805
Changed lines of the file:
@@
 F 0 "U1" H 7400 4150 50  0000 L CNN
 F 1 "LM358N" H 7400 3700 50  0000 L CNN
-F 2 "SMD_Packages:SOIC-8-N" H 7450 3950 50  0001 C CNN
+F 2 "lib_fp:SOIC-8-N" H 7450 3950 50  0001 C CNN
 F 3 "" H 7450 3950 50  0000 C CNN
 	1    7450 3950
@@
 F 0 "U12" H 4900 4050 60  0000 C CNN
 F 1 "TCRT5000" H 4850 4150 60  0000 C CNN
-F 2 "cyclophone:TCRT5000" H 5550 4800 60  0001 C CNN
+F 2 "lib_fp:TCRT5000" H 5550 4800 60  0001 C CNN
 F 3 "" H 5550 4800 60  0000 C CNN
 	1    4700 3900
@@
 F 0 "U5" V 4050 3250 50  0000 C CNN
 F 1 "20K" V 3850 3450 50  0000 C CNN
-F 2 "Resistors_SMD:R_0805" V 3830 3250 50  0001 C CNN
+F 2 "lib_fp:R_0805" V 3830 3250 50  0001 C CNN
 F 3 "" H 3900 3250 50  0000 C CNN
 	1    3900 3250
@@
 F 0 "U13" V 5430 3250 50  0000 C CNN
 F 1 "100R" V 5350 3400 50  0000 C CNN
-F 2 "Resistors_SMD:R_0805" V 5280 3250 50  0001 C CNN
+F 2 "lib_fp:R_0805" V 5280 3250 50  0001 C CNN
 F 3 "" H 5350 3250 50  0000 C CNN
 	1    5350 3250
@@
 F 0 "U7" H 6000 2700 50  0000 C CNN
 F 1 "10k" H 6000 2800 50  0000 C CNN
-F 2 "Potentiometers:Potentiometer_Trimmer_Bourns_3296W" H 6000 2800 50  0001 C CNN
+F 2 "lib_fp:Potentiometer_Trimmer_Bourns_3296W" H 6000 2800 50  0001 C CNN
 F 3 "" H 6000 2800 50  0000 C CNN
 	1    6000 2800
@@
 F 0 "U6" V 6530 3200 50  0000 C CNN
 F 1 "10K" V 6450 3350 50  0000 C CNN
-F 2 "Resistors_SMD:R_0805" V 6380 3200 50  0001 C CNN
+F 2 "lib_fp:R_0805" V 6380 3200 50  0001 C CNN
 F 3 "" H 6450 3200 50  0000 C CNN
 	1    6450 3200
@@
 F 0 "U9" H 7950 3300 50  0000 C CNN
 F 1 "LED" H 7950 3100 50  0000 C CNN
-F 2 "LEDs:LED_0805" H 7950 3200 50  0001 C CNN
+F 2 "lib_fp:LED_0805" H 7950 3200 50  0001 C CNN
 F 3 "" H 7950 3200 50  0000 C CNN
 	1    7950 3200
@@
 F 0 "U3" V 8030 3650 50  0000 C CNN
 F 1 "1K" V 7950 3750 50  0000 C CNN
-F 2 "Resistors_SMD:R_0805" V 7880 3650 50  0001 C CNN
+F 2 "lib_fp:R_0805" V 7880 3650 50  0001 C CNN
 F 3 "" H 7950 3650 50  0000 C CNN
 	1    7950 3650
@@
 F 0 "U10" H 8475 3250 50  0000 L CNN
 F 1 "100nF" H 8475 3050 50  0000 L CNN
-F 2 "Resistors_SMD:R_0805" H 8488 3000 50  0001 C CNN
+F 2 "lib_fp:R_0805" H 8488 3000 50  0001 C CNN
 F 3 "" H 8450 3150 50  0000 C CNN
 	1    8450 3150
@@
 F 0 "U8" H 9200 4050 50  0000 C CNN
 F 1 "CON3_ET" V 9300 3850 50  0000 C CNN
-F 2 "Connectors_JST:JST_PH_S3B-PH-K_03x2.00mm_Angled" H 9200 3850 50  0001 C CNN
+F 2 "lib_fp:JST_PH_S3B-PH-K_03x2.00mm_Angled" H 9200 3850 50  0001 C CNN
 F 3 "" H 9200 3850 50  0000 C CNN
 	1    9200 3850
